File: KiCad_Files/spaceEggs.kicad_pcb (KiCad board)
At the start: 2 copper layers, 45 x 45 mm, 7 parts, among them SW1 SW_Reed

Commit message: closing Issue #2
Parts:
- added ce-symbol_mask_3mm: G***, blinkyparts:ce-icon_3mm, F.Cu at (108.0, 78.1)
- added weee-symbol_mask_3mm: G***, blinkyparts:weee-icon_3mm, F.Cu at (113.1, 78.1)
Other:
- board text added: "blinkyparts GmbH Egerstr. 9 93057 Regensburg blinkyparts.com"

Commit message: some changes and added bom
Parts:
- moved ce-symbol_mask_3mm 28.5 mm to (107.5, 49.6)
- moved weee-symbol_mask_3mm 25.4 mm to (108.6, 53.1)
Other:
- board text added: "v1.2"
- board text removed: "Manual: LEDs: Long leg is + (anode) LED-Head sticks out at the white circle 1. Solder LED1 first 2. Solder LED2 and LED3 3. LED4 and LED5 are optional. 4. Solder SW1 reed contact 5. Solder battery holder"
- board text removed: "v1.1"
