File: KiCad_Files/spaceEggs.kicad_sch (KiCad schematic)
At the start: 7 parts, among them SW1 SW_Reed

Commit message: some changes and added bom
Changed lines of the file:
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@@
 (kicad_sch
-	(version 20231120)
+	(version 20250114)
 	(generator "eeschema")
-	(generator_version "8.0")
+	(generator_version "9.0")
 	(paper "A4")
 	(junction
@@
 		)
 	)
+	(embedded_fonts no)
 )
